File: pcb/6_buttons.kicad_pcb (KiCad board)
At the start: 2 copper layers, 92.5 x 55.5 mm, 18 parts, among them SW1 SW_Push, SW2 SW_Push, SW3 SW_Push, SW4 SW_Push, SW5 SW_Push, SW6 SW_Push, SW7 RotaryEncoder, U1 XIAO-RP2040-DIP

Commit message: update gerb
Parts:
- moved U1 5.79 mm to (204.0, 93.0)
Routing:
- net COLUMN 3: track 58.8 -> 66.4 mm
- net SIGNAL B: track 29.1 -> 36.3 mm
- net SIGNAL A: track 40.7 -> 47.8 mm
- net COLUMN 1: track 110.2 -> 115.5 mm
- net ROW 1: track 67.4 -> 72.3 mm
- net ROW 2: track 60.7 -> 56.2 mm
- net GND: track 40.4 -> 44.2 mm
- net COLUMN 2: track 91.8 -> 88.4 mm
- net unconnected-(U1-GPIO7/SCL-Pad6): track 0.00 -> 1.08 mm
Changed lines of the file:
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@@
 			(outputformat 1)
 			(mirror no)
-			(drillshape 1)
+			(drillshape 0)
 			(scaleselection 1)
-			(outputdirectory "")
+			(outputdirectory "../../../../Downloads/gerb/")
 		)
 	)
@@
 	(footprint "Seeed Studio XIAO Series Library:XIAO-RP2040-DIP"
 		(layer "F.Cu")
-		(at 204.5 87.2315 180)
+		(at 204 93 180)
 		(property "Reference" "U1"
 			(at -8.5 -12 180)
@@
 	)
 	(segment
-		(start 196.88 79.6115)
-		(end 195.6115 79.6115)
+		(start 191 75)
+		(end 196.38 80.38)
 		(width 0.2)
 		(layer "F.Cu")
@@
 	)
 	(segment
-		(start 191 59.19)
-		(end 187.81 56)
+		(start 196.38 80.38)
+		(end 196.38 85.38)
 		(width 0.2)
 		(layer "F.Cu")
@@
 	)
 	(segment
-		(start 191 75)
-		(end 191 59.19)
+		(start 191 59.19)
+		(end 187.81 56)
 		(width 0.2)
 		(layer "F.Cu")
@@
 	)
 	(segment
-		(start 195.6115 79.6115)
-		(end 191 75)
+		(start 191 75)
+		(end 191 59.19)
 		(width 0.2)
 		(layer "F.Cu")
@@
 	)
 	(segment
-		(start 196.045 82.1515)
-		(end 196.88 82.1515)
+		(start 193.08 87.92)
+		(end 196.38 87.92)
 		(width 0.2)
 		(layer "F.Cu")
@@
 	)
 	(segment
-		(start 188.81 89.3865)
-		(end 196.045 82.1515)
+		(start 188.81 98.5)
+		(end 188.81 96.69)
 		(width 0.2)
 		(layer "F.Cu")
@@
 	)
 	(segment
-		(start 188.81 98.5)
-		(end 188.81 89.3865)
+		(start 192 89)
+		(end 193.08 87.92)
+		(width 0.2)
+		(layer "F.Cu")
+		(net 5)
+	)
+	(segment
+		(start 192 93.5)
+		(end 192 89)
+		(width 0.2)
+		(layer "F.Cu")
+		(net 5)
+	)
+	(segment
+		(start 188.81 96.69)
+		(end 192 93.5)
 		(width 0.2)
 		(layer "F.Cu")
@@
 	)
 	(segment
-		(start 168.04 81.46)
-		(end 173.96 81.46)
+		(start 215 98.5)
+		(end 214.5 98)
 		(width 0.2)
 		(layer "B.Cu")
@@
 	)
 	(segment
-		(start 215.5 93.5)
-		(end 214.3115 92.3115)
+		(start 215 100.5)
+		(end 215 98.5)
 		(width 0.2)
 		(layer "B.Cu")
@@
 	)
 	(segment
-		(start 173.96 81.46)
-		(end 175.5 83)
+		(start 193.5 97)
+		(end 203.9329 97)
 		(width 0.2)
 		(layer "B.Cu")
@@
 	)
 	(segment
-		(start 215.5 97.5)
-		(end 215.5 93.5)
+		(start 168.04 81.46)
+		(end 173.96 81.46)
+		(width 0.2)
+		(layer "B.Cu")
+		(net 9)
+	)
+	(segment
+		(start 173.96 81.46)
+		(end 175.5 83)
 		(width 0.2)
 		(layer "B.Cu")
@@
 	)
 	(segment
-		(start 197.5 101)
-		(end 212 101)
+		(start 214.5 98)
+		(end 214.42 98.08)
 		(width 0.2)
 		(layer "B.Cu")
@@
 	)
 	(segment
-		(start 193 96.5)
-		(end 197.5 101)
+		(start 208.6159 101.683)
+		(end 213.817 101.683)
 		(width 0.2)
 		(layer "B.Cu")
@@
 	)
 	(segment
-		(start 214.3115 92.3115)
-		(end 212.12 92.3115)
+		(start 214.42 98.08)
+		(end 211.62 98.08)
 		(width 0.2)
 		(layer "B.Cu")
@@
 	)
 	(segment
-		(start 212 101)
-		(end 215.5 97.5)
+		(start 203.9329 97)
+		(end 208.6159 101.683)
+		(width 0.2)
+		(layer "B.Cu")
+		(net 9)
+	)
+	(segment
+		(start 213.817 101.683)
+		(end 215 100.5)
+		(width 0.2)
+		(layer "B.Cu")
+		(net 9)
+	)
+	(segment
+		(start 193 96.5)
+		(end 193.5 97)
 		(width 0.2)
 		(layer "B.Cu")
@@
 	)
 	(segment
-		(start 205 87.7315)
-		(end 205 77.5)
+		(start 205 97.5)
+		(end 208.12 100.62)
 		(width 0.2)
 		(layer "B.Cu")
@@
 	(segment
 		(start 205 77.5)
-		(end 190.96 77.5)
+		(end 205 97.5)
 		(width 0.2)
 		(layer "B.Cu")
@@
 	)
 	(segment
-		(start 190.96 77.5)
-		(end 187.04 81.42)
+		(start 208.12 100.62)
+		(end 211.62 100.62)
 		(width 0.2)
 		(layer "B.Cu")
@@
 	)
 	(segment
-		(start 212.12 94.8515)
-		(end 205 87.7315)
+		(start 187.04 81.42)
+		(end 190.96 77.5)
+		(width 0.2)
+		(layer "B.Cu")
+		(net 10)
+	)
+	(segment
+		(start 190.96 77.5)
+		(end 205 77.5)
 		(width 0.2)
 		(layer "B.Cu")
@@
 	)
 	(segment
-		(start 216.7285 89.7715)
-		(end 212.12 89.7715)
+		(start 214.96 95.54)
+		(end 211.62 95.54)
 		(width 0.2)
 		(layer "B.Cu")
@@
 	)
 	(segment
-		(start 155.5 75)
-		(end 216.5 75)
+		(start 216.5 75)
+		(end 218.5 77)
 		(width 0.2)
 		(layer "B.Cu")
@@
 	)
 	(segment
-		(start 218.5 88)
-		(end 216.7285 89.7715)
+		(start 218.5 92)
+		(end 214.96 95.54)
 		(width 0.2)
 		(layer "B.Cu")
@@
 	)
 	(segment
-		(start 149 81.5)
-		(end 155.5 75)
+		(start 218.5 77)
+		(end 218.5 92)
 		(width 0.2)
 		(layer "B.Cu")
@@
 	)
 	(segment
-		(start 216.5 75)
-		(end 218.5 77)
+		(start 155.5 75)
+		(end 216.5 75)
 		(width 0.2)
 		(layer "B.Cu")
@@
 	)
 	(segment
-		(start 218.5 77)
-		(end 218.5 88)
+		(start 149 81.5)
+		(end 155.5 75)
 		(width 0.2)
 		(layer "B.Cu")
@@
 	)
 	(segment
-		(start 195.5 68.0715)
-		(end 212.12 84.6915)
+		(start 195.5 68)
+		(end 207.5 80)
+		(width 0.2)
+		(layer "F.Cu")
+		(net 12)
+	)
+	(segment
+		(start 208.96 90.46)
+		(end 211.62 90.46)
 		(width 0.2)
 		(layer "F.Cu")
@@
 	(segment
 		(start 195.5 62.5)
+		(end 195.5 68)
+		(width 0.2)
+		(layer "F.Cu")
+		(net 12)
+	)
+	(segment
+		(start 195.5 68)
 		(end 195.5 68.0715)
 		(width 0.2)
@@
 	)
 	(segment
-		(start 198.102 57.5)
-		(end 195.5 57.5)
+		(start 207.5 80)
+		(end 207.5 89)
+		(width 0.2)
+		(layer "F.Cu")
+		(net 12)
+	)
+	(segment
+		(start 207.5 89)
+		(end 208.96 90.46)
+		(width 0.2)
+		(layer "F.Cu")
+		(net 12)
+	)
+	(segment
+		(start 214.472 92.972)
+		(end 214.5 93)
 		(width 0.2)
 		(layer "F.Cu")
@@
 	)
 	(segment
-		(start 214.472 85.95713)
+		(start 198.102 57.5)
 		(end 214.472 73.87)
 		(width 0.2)
@@
 	)
 	(segment
-		(start 214.472 73.87)
+		(start 195.5 57.5)
 		(end 198.102 57.5)
 		(width 0.2)
@@
 	)
 	(segment
-		(start 213.19763 87.2315)
-		(end 214.472 85.95713)
+		(start 214.472 73.87)
+		(end 214.472 92.972)
 		(width 0.2)
 		(layer "F.Cu")
@@
 	)
 	(segment
-		(start 212.12 87.2315)
-		(end 213.19763 87.2315)
+		(start 214.5 93)
+		(end 211.62 93)
 		(width 0.2)
 		(layer "F.Cu")
@@
 	)
 	(segment
-		(start 199.5 92)
-		(end 199.5 76.5)
+		(start 195.5 60)
+		(end 193.5 62)
 		(width 0.2)
 		(layer "F.Cu")
@@
 	)
 	(segment
-		(start 193.5 62)
-		(end 195.5 60)
+		(start 193.5 73)
+		(end 196.5 76)
 		(width 0.2)
 		(layer "F.Cu")
@@
 	)
 	(segment
-		(start 196.5 76)
-		(end 193.5 73)
+		(start 199.5 76.5)
+		(end 199.5 94.96)
 		(width 0.2)
 		(layer "F.Cu")
@@
 	)
 	(segment
-		(start 193.5 73)
-		(end 193.5 62)
+		(start 199 76)
+		(end 199.5 76.5)
 		(width 0.2)
 		(layer "F.Cu")
@@
 	)
 	(segment
-		(start 199.5 76.5)
-		(end 199 76)
+		(start 199.5 94.96)
+		(end 196.38 98.08)
 		(width 0.2)
 		(layer "F.Cu")
@@
 	)
 	(segment
-		(start 199 76)
-		(end 196.5 76)
+		(start 193.5 62)
+		(end 193.5 73)
 		(width 0.2)
 		(layer "F.Cu")
@@
 	)
 	(segment
-		(start 199.1885 92.3115)
-		(end 199.5 92)
+		(start 196.5 76)
+		(end 199 76)
 		(width 0.2)
 		(layer "F.Cu")
@@
 	)
 	(segment
-		(start 196.045 92.3115)
-		(end 199.1885 92.3115)
+		(start 212.12 87.2315)
+		(end 213.19763 87.2315)
 		(width 0.2)
 		(layer "F.Cu")
-		(net 14)
+		(net 19)
 	)
 	(embedded_fonts no)
